File: Codec.kicad_sch (KiCad schematic)
At the start: 17 parts, among them U8 CS4272

Commit message: Buffer and layout
Updated the input and output buffers.
Updated the board layout.
Parts:
- C33: renamed from C46; value 4.7u -> 10u
- C37: renamed from C50; value 4.7u -> 10u
- renumbered C42 to C29, C43 to C30, C44 to C31, C45 to C32, C47 to C34, C48 to C35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
Connections:
- net VFILT+ renamed FILT+
