File: SimpleCodec.kicad_pcb (KiCad board)
At the start: 4 copper layers, 59 x 95 mm, 99 parts, among them J1 RPI_ADC, J2 RP_GPIO, U1 AMS1117-5.0, U2 AMS1117-3.3, U3 MCP6002-xSN, U4 MCP6002-xSN, U5 CS4272, X1 PEDAL_COMBO_TOP

Commit message: Via stitching
Added missing vias to GND.
Routing:
- net VCOM: track 88.6 -> 86.0 mm
- net GND: vias 260 -> 289
