File: Hardware/Buffers_In.kicad_sch (KiCad schematic)
At the start: 19 parts, among them U3 MCP6002-xSN, X1 PEDAL_COMBO_TOP

Commit message: Layout review
Updated the LDO layout to include a series resistor for stability.
Updated all build files.
Parts:
- renumbered R8 to R10, R9 to R11, R10 to R12, R3 to R5, R4 to R6, R5 to R7, R6 to R8, R7 to R9
Changed lines of the file:
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@@
 		(dnp no)
 		(fields_autoplaced yes)
-		(property "Reference" "R9"
+		(property "Reference" "R11"
 			(at 176.53 48.26 90)
 			(show_name no)
@@
 			(project "PicoFX"
 				(path "/4cbf131b-42e8-4a05-beea-68c6d66cdb1a/469e8ad1-854f-4ea5-8b66-be90c8cb100f"
-					(reference "R9")
+					(reference "R11")
 					(unit 1)
 				)
@@
 		(dnp no)
 		(fields_autoplaced yes)
-		(property "Reference" "R5"
+		(property "Reference" "R7"
 			(at 134.62 57.1499 0)
 			(show_name no)
@@
 			(project "PicoFX"
 				(path "/4cbf131b-42e8-4a05-beea-68c6d66cdb1a/469e8ad1-854f-4ea5-8b66-be90c8cb100f"
-					(reference "R5")
+					(reference "R7")
 					(unit 1)
 				)
@@
 		(dnp no)
 		(fields_autoplaced yes)
-		(property "Reference" "R10"
+		(property "Reference" "R12"
 			(at 176.53 118.11 90)
 			(show_name no)
@@
 			(project "PicoFX"
 				(path "/4cbf131b-42e8-4a05-beea-68c6d66cdb1a/469e8ad1-854f-4ea5-8b66-be90c8cb100f"
-					(reference "R10")
+					(reference "R12")
 					(unit 1)
 				)
@@
 		(dnp no)
 		(fields_autoplaced yes)
-		(property "Reference" "R6"
+		(property "Reference" "R8"
 			(at 134.62 126.9999 0)
 			(show_name no)
@@
 			(project "PicoFX"
 				(path "/4cbf131b-42e8-4a05-beea-68c6d66cdb1a/469e8ad1-854f-4ea5-8b66-be90c8cb100f"
-					(reference "R6")
+					(reference "R8")
 					(unit 1)
 				)
@@
 		(dnp no)
 		(fields_autoplaced yes)
-		(property "Reference" "R8"
+		(property "Reference" "R10"
 			(at 152.4 111.7599 0)
 			(show_name no)
@@
 			(project "PicoFX"
 				(path "/4cbf131b-42e8-4a05-beea-68c6d66cdb1a/469e8ad1-854f-4ea5-8b66-be90c8cb100f"
-					(reference "R8")
+					(reference "R10")
 					(unit 1)
 				)
@@
 		(dnp no)
 		(fields_autoplaced yes)
-		(property "Reference" "R4"
+		(property "Reference" "R6"
 			(at 115.57 115.57 90)
 			(show_name no)
@@
 			(project "PicoFX"
 				(path "/4cbf131b-42e8-4a05-beea-68c6d66cdb1a/469e8ad1-854f-4ea5-8b66-be90c8cb100f"
-					(reference "R4")
+					(reference "R6")
 					(unit 1)
 				)
@@
 		(dnp no)
 		(fields_autoplaced yes)
-		(property "Reference" "R7"
+		(property "Reference" "R9"
 			(at 152.4 41.9099 0)
 			(show_name no)
@@
 			(project "PicoFX"
 				(path "/4cbf131b-42e8-4a05-beea-68c6d66cdb1a/469e8ad1-854f-4ea5-8b66-be90c8cb100f"
-					(reference "R7")
+					(reference "R9")
 					(unit 1)
 				)
@@
 		(dnp no)
 		(fields_autoplaced yes)
-		(property "Reference" "R3"
+		(property "Reference" "R5"
 			(at 115.57 45.72 90)
 			(show_name no)
@@
 			(project "PicoFX"
 				(path "/4cbf131b-42e8-4a05-beea-68c6d66cdb1a/469e8ad1-854f-4ea5-8b66-be90c8cb100f"
-					(reference "R3")
-					(unit 1)
-				)
+					(reference "R5")
+					(unit 1)
+				)

Commit message: Output files
Updated the board silkscreen.
Upddated the output files.
Parts:
- C15, C16, C19, C20: JLCPCB Part (none) -> C28260; Manufacturer Part (none) -> CL21C222JBFNNNE
- C17, C18: JLCPCB Part (none) -> C15850; Manufacturer Part (none) -> CL21A106KAYNNNE
- C21: JLCPCB Part (none) -> C14663; Manufacturer Part (none) -> CC0603KRX7R9BB104
- D3, D4: JLCPCB Part (none) -> C20615814; Manufacturer Part (none) -> H15VSD3B
- R10, R7, R8, R9: JLCPCB Part (none) -> C22935; Manufacturer Part (none) -> 0603WAF1004T5E
- R11, R12: JLCPCB Part (none) -> C21190; Manufacturer Part (none) -> 0603WAF1001T5E
- R5, R6: JLCPCB Part (none) -> C22775; Manufacturer Part (none) -> 0603WAF1000T5E
- U3: JLCPCB Part (none) -> C7377; Manufacturer Part (none) -> MCP6002T-I/SN
- X1: now left out of the parts list

Commit message: Assembly review
Performed a full review of the schematic and layout.
Minor changes to the schematic and layout.
Updated output files.
Parts:
- X1: JLCPCB Part (none) -> -; Manufacturer Part (none) -> -
Changed lines of the file:
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@@
+			)
+		)
+		(property "JLCPCB Part" "-"
+			(at 50.8 88.9 0)
+			(hide yes)
+			(show_name no)
+			(do_not_autoplace no)
+			(effects
+				(font
+					(size 1.27 1.27)
+				)
+			)
+		)
+		(property "Manufacturer Part" "-"
+			(at 50.8 88.9 0)
+			(hide yes)
+			(show_name no)
+			(do_not_autoplace no)
+			(effects
+				(font
+					(size 1.27 1.27)
+				)
 			)
 		)
