File: Hardware/Buffers_Out.kicad_sch (KiCad schematic)
At the start: 29 parts, among them U4 MCP6002-xSN, X1 PEDAL_COMBO_TOP

Commit message: Name update
Updated the name of the project.
Updated the silkscreen for the PCB layout.
Other:
- title: SIMPLE CODEC -> PICO FX
Changed lines of the file:
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@@
 	(paper "A4")
 	(title_block
-		(title "SIMPLE CODEC")
+		(title "PICO FX")
 		(date "2026-04-08")
 		(rev "1.0")
@@
 		)
 		(instances
-			(project "SimpleCodec"
+			(project "PicoFX"
 				(path "/4cbf131b-42e8-4a05-beea-68c6d66cdb1a/f30b69e3-f4a5-44b3-bff9-cd489323ac3e"
 					(reference "R16")
@@
 		)
 		(instances
-			(project "SimpleCodec"
+			(project "PicoFX"
 				(path "/4cbf131b-42e8-4a05-beea-68c6d66cdb1a/f30b69e3-f4a5-44b3-bff9-cd489323ac3e"
 					(reference "R14")
@@
 		)
 		(instances
-			(project "SimpleCodec"
+			(project "PicoFX"
 				(path "/4cbf131b-42e8-4a05-beea-68c6d66cdb1a/f30b69e3-f4a5-44b3-bff9-cd489323ac3e"
 					(reference "C18")
@@
 		)
 		(instances
-			(project "SimpleCodec"
+			(project "PicoFX"
 				(path "/4cbf131b-42e8-4a05-beea-68c6d66cdb1a/f30b69e3-f4a5-44b3-bff9-cd489323ac3e"
 					(reference "#PWR039")
@@
 		)
 		(instances
-			(project "SimpleCodec"
+			(project "PicoFX"
 				(path "/4cbf131b-42e8-4a05-beea-68c6d66cdb1a/f30b69e3-f4a5-44b3-bff9-cd489323ac3e"
 					(reference "#PWR040")
@@
 		)
 		(instances
-			(project "SimpleCodec"
+			(project "PicoFX"
 				(path "/4cbf131b-42e8-4a05-beea-68c6d66cdb1a/f30b69e3-f4a5-44b3-bff9-cd489323ac3e"
 					(reference "U4")
@@
 		)
 		(instances
-			(project "SimpleCodec"
+			(project "PicoFX"
 				(path "/4cbf131b-42e8-4a05-beea-68c6d66cdb1a/f30b69e3-f4a5-44b3-bff9-cd489323ac3e"
 					(reference "R26")
@@
 		)
 		(instances
-			(project "SimpleCodec"
+			(project "PicoFX"
 				(path "/4cbf131b-42e8-4a05-beea-68c6d66cdb1a/f30b69e3-f4a5-44b3-bff9-cd489323ac3e"
 					(reference "#PWR038")
@@
 		)
 		(instances
-			(project "SimpleCodec"
+			(project "PicoFX"
 				(path "/4cbf131b-42e8-4a05-beea-68c6d66cdb1a/f30b69e3-f4a5-44b3-bff9-cd489323ac3e"
 					(reference "R21")
@@
 		)
 		(instances
-			(project "SimpleCodec"
+			(project "PicoFX"
 				(path "/4cbf131b-42e8-4a05-beea-68c6d66cdb1a/f30b69e3-f4a5-44b3-bff9-cd489323ac3e"
 					(reference "D6")
@@
 		)
 		(instances
-			(project "SimpleCodec"
+			(project "PicoFX"
 				(path "/4cbf131b-42e8-4a05-beea-68c6d66cdb1a/f30b69e3-f4a5-44b3-bff9-cd489323ac3e"
 					(reference "D5")
@@
 		)
 		(instances
-			(project "SimpleCodec"
+			(project "PicoFX"
 				(path "/4cbf131b-42e8-4a05-beea-68c6d66cdb1a/f30b69e3-f4a5-44b3-bff9-cd489323ac3e"
 					(reference "#PWR044")
@@
 		)
 		(instances
-			(project "SimpleCodec"
+			(project "PicoFX"
 				(path "/4cbf131b-42e8-4a05-beea-68c6d66cdb1a/f30b69e3-f4a5-44b3-bff9-cd489323ac3e"
 					(reference "#PWR042")
@@
 		)
 		(instances
-			(project "SimpleCodec"
+			(project "PicoFX"
 				(path "/4cbf131b-42e8-4a05-beea-68c6d66cdb1a/f30b69e3-f4a5-44b3-bff9-cd489323ac3e"
 					(reference "#PWR043")
@@
 		)
 		(instances
-			(project "SimpleCodec"
+			(project "PicoFX"
 				(path "/4cbf131b-42e8-4a05-beea-68c6d66cdb1a/f30b69e3-f4a5-44b3-bff9-cd489323ac3e"
 					(reference "C19")
@@
 		)
 		(instances
-			(project "SimpleCodec"
+			(project "PicoFX"
 				(path "/4cbf131b-42e8-4a05-beea-68c6d66cdb1a/f30b69e3-f4a5-44b3-bff9-cd489323ac3e"
 					(reference "X1")
@@
 		)
 		(instances
-			(project "SimpleCodec"
+			(project "PicoFX"
 				(path "/4cbf131b-42e8-4a05-beea-68c6d66cdb1a/f30b69e3-f4a5-44b3-bff9-cd489323ac3e"
 					(reference "U4")
@@
 		)
 		(instances
-			(project "SimpleCodec"
+			(project "PicoFX"
 				(path "/4cbf131b-42e8-4a05-beea-68c6d66cdb1a/f30b69e3-f4a5-44b3-bff9-cd489323ac3e"
 					(reference "R12")
@@
 		)
 		(instances
-			(project "SimpleCodec"
+			(project "PicoFX"
 				(path "/4cbf131b-42e8-4a05-beea-68c6d66cdb1a/f30b69e3-f4a5-44b3-bff9-cd489323ac3e"
 					(reference "C26")
@@
 		)
 		(instances
-			(project "SimpleCodec"
+			(project "PicoFX"
 				(path "/4cbf131b-42e8-4a05-beea-68c6d66cdb1a/f30b69e3-f4a5-44b3-bff9-cd489323ac3e"
 					(reference "R15")
@@
 		)
 		(instances
-			(project "SimpleCodec"
+			(project "PicoFX"
 				(path "/4cbf131b-42e8-4a05-beea-68c6d66cdb1a/f30b69e3-f4a5-44b3-bff9-cd489323ac3e"
 					(reference "R18")
@@
 		)
 		(instances
-			(project "SimpleCodec"
+			(project "PicoFX"
 				(path "/4cbf131b-42e8-4a05-beea-68c6d66cdb1a/f30b69e3-f4a5-44b3-bff9-cd489323ac3e"
 					(reference "C24")
@@
 		)
 		(instances
-			(project "SimpleCodec"
+			(project "PicoFX"
 				(path "/4cbf131b-42e8-4a05-beea-68c6d66cdb1a/f30b69e3-f4a5-44b3-bff9-cd489323ac3e"
 					(reference "C20")
@@
 		)
 		(instances
-			(project "SimpleCodec"
+			(project "PicoFX"
 				(path "/4cbf131b-42e8-4a05-beea-68c6d66cdb1a/f30b69e3-f4a5-44b3-bff9-cd489323ac3e"
 					(reference "R20")
@@
 		)
 		(instances
-			(project "SimpleCodec"
+			(project "PicoFX"
 				(path "/4cbf131b-42e8-4a05-beea-68c6d66cdb1a/f30b69e3-f4a5-44b3-bff9-cd489323ac3e"
 					(reference "R25")
@@
 		)
 		(instances
-			(project "SimpleCodec"
+			(project "PicoFX"
 				(path "/4cbf131b-42e8-4a05-beea-68c6d66cdb1a/f30b69e3-f4a5-44b3-bff9-cd489323ac3e"
 					(reference "R17")
@@
 		)
 		(instances
-			(project "SimpleCodec"
+			(project "PicoFX"
 				(path "/4cbf131b-42e8-4a05-beea-68c6d66cdb1a/f30b69e3-f4a5-44b3-bff9-cd489323ac3e"
 					(reference "C25")
@@
 		)
 		(instances
-			(project "SimpleCodec"
+			(project "PicoFX"
 				(path "/4cbf131b-42e8-4a05-beea-68c6d66cdb1a/f30b69e3-f4a5-44b3-bff9-cd489323ac3e"
 					(reference "R22")
@@
 		)
 		(instances
-			(project "SimpleCodec"
+			(project "PicoFX"
 				(path "/4cbf131b-42e8-4a05-beea-68c6d66cdb1a/f30b69e3-f4a5-44b3-bff9-cd489323ac3e"
 					(reference "U4")
@@
 		)
 		(instances
-			(project "SimpleCodec"
+			(project "PicoFX"
 				(path "/4cbf131b-42e8-4a05-beea-68c6d66cdb1a/f30b69e3-f4a5-44b3-bff9-cd489323ac3e"
 					(reference "C21")
@@
 		)
 		(instances
-			(project "SimpleCodec"
+			(project "PicoFX"
 				(path "/4cbf131b-42e8-4a05-beea-68c6d66cdb1a/f30b69e3-f4a5-44b3-bff9-cd489323ac3e"
 					(reference "R13")
@@
 		)
 		(instances
-			(project "SimpleCodec"
+			(project "PicoFX"
 				(path "/4cbf131b-42e8-4a05-beea-68c6d66cdb1a/f30b69e3-f4a5-44b3-bff9-cd489323ac3e"
 					(reference "R24")
@@
 		)
 		(instances
-			(project "SimpleCodec"
+			(project "PicoFX"
 				(path "/4cbf131b-42e8-4a05-beea-68c6d66cdb1a/f30b69e3-f4a5-44b3-bff9-cd489323ac3e"
 					(reference "C23")
@@
 		)
 		(instances
-			(project "SimpleCodec"
+			(project "PicoFX"
 				(path "/4cbf131b-42e8-4a05-beea-68c6d66cdb1a/f30b69e3-f4a5-44b3-bff9-cd489323ac3e"
 					(reference "R23")
@@
 		)
 		(instances
-			(project "SimpleCodec"
+			(project "PicoFX"
 				(path "/4cbf131b-42e8-4a05-beea-68c6d66cdb1a/f30b69e3-f4a5-44b3-bff9-cd489323ac3e"
 					(reference "R19")
@@
 		)
 		(instances
-			(project "SimpleCodec"
+			(project "PicoFX"
 				(path "/4cbf131b-42e8-4a05-beea-68c6d66cdb1a/f30b69e3-f4a5-44b3-bff9-cd489323ac3e"
 					(reference "#PWR041")
@@
 		)
 		(instances
-			(project "SimpleCodec"
+			(project "PicoFX"
 				(path "/4cbf131b-42e8-4a05-beea-68c6d66cdb1a/f30b69e3-f4a5-44b3-bff9-cd489323ac3e"
 					(reference "C22")
@@
 		)
 		(instances
-			(project "SimpleCodec"
+			(project "PicoFX"
 				(path "/4cbf131b-42e8-4a05-beea-68c6d66cdb1a/f30b69e3-f4a5-44b3-bff9-cd489323ac3e"
 					(reference "#PWR045")
@@
 		)
 		(instances
-			(project "SimpleCodec"
+			(project "PicoFX"
 				(path "/4cbf131b-42e8-4a05-beea-68c6d66cdb1a/f30b69e3-f4a5-44b3-bff9-cd489323ac3e"
 					(reference "#PWR046")
@@
 		)
 		(instances
-			(project "SimpleCodec"
+			(project "PicoFX"
 				(path "/4cbf131b-42e8-4a05-beea-68c6d66cdb1a/f30b69e3-f4a5-44b3-bff9-cd489323ac3e"
 					(reference "R11")
