File: Hardware/Codec.kicad_sch (KiCad schematic)
At the start: 17 parts, among them U5 CS4272

Commit message: Layout review
Updated the LDO layout to include a series resistor for stability.
Updated all build files.
Parts:
- renumbered R27 to R29, R28 to R30, R29 to R31, R30 to R32
Changed lines of the file:
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@@
 		(dnp no)
 		(fields_autoplaced yes)
-		(property "Reference" "R29"
+		(property "Reference" "R31"
 			(at 180.34 102.8699 0)
 			(show_name no)
@@
 			(project "PicoFX"
 				(path "/4cbf131b-42e8-4a05-beea-68c6d66cdb1a/f7920eb9-f1f4-4882-8d74-32484732cce5"
-					(reference "R29")
+					(reference "R31")
 					(unit 1)
 				)
@@
 		(in_pos_files yes)
 		(dnp no)
-		(property "Reference" "R28"
+		(property "Reference" "R30"
 			(at 100.33 105.4099 0)
 			(show_name no)
@@
 			(project "PicoFX"
 				(path "/4cbf131b-42e8-4a05-beea-68c6d66cdb1a/f7920eb9-f1f4-4882-8d74-32484732cce5"
-					(reference "R28")
+					(reference "R30")
 					(unit 1)
 				)
@@
 		(dnp no)
 		(fields_autoplaced yes)
-		(property "Reference" "R30"
+		(property "Reference" "R32"
 			(at 190.5 102.8699 0)
 			(show_name no)
@@
 			(project "PicoFX"
 				(path "/4cbf131b-42e8-4a05-beea-68c6d66cdb1a/f7920eb9-f1f4-4882-8d74-32484732cce5"
-					(reference "R30")
+					(reference "R32")
 					(unit 1)
 				)
@@
 		(in_pos_files yes)
 		(dnp no)
-		(property "Reference" "R27"
+		(property "Reference" "R29"
 			(at 91.44 105.4099 0)
 			(show_name no)
@@
 			(project "PicoFX"
 				(path "/4cbf131b-42e8-4a05-beea-68c6d66cdb1a/f7920eb9-f1f4-4882-8d74-32484732cce5"
-					(reference "R27")
-					(unit 1)
-				)
+					(reference "R29")
+					(unit 1)
+				)

Commit message: Output files
Updated the board silkscreen.
Upddated the output files.
Parts:
- C31, C32, C40, C41: JLCPCB Part (none) -> C28323; Manufacturer Part (none) -> CL21B105KBFNNNE
- C33, C34, C36, C37, C38: JLCPCB Part (none) -> C14663; Manufacturer Part (none) -> CC0603KRX7R9BB104
- C35, C39: JLCPCB Part (none) -> C28260; Manufacturer Part (none) -> CL21C222JBFNNNE
- C42: JLCPCB Part (none) -> C15850; Manufacturer Part (none) -> CL21A106KAYNNNE
- R29, R30, R31, R32: JLCPCB Part (none) -> C25819; Manufacturer Part (none) -> 0603WAF4702T5E
- U5: JLCPCB Part (none) -> C2151111; Manufacturer Part (none) -> CS4272-CZZR

Commit message: Assembly review
Performed a full review of the schematic and layout.
Minor changes to the schematic and layout.
Updated output files.
Parts:
- R29, R30: value 47K -> 2.2K; JLCPCB Part C25819 -> C4190; Manufacturer Part 0603WAF4702T5E -> 0603WAF2201T5E
Changed lines of the file:
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@@
 			)
 		)
-		(property "Value" "47K"
+		(property "Value" "2.2K"
 			(at 100.33 107.9499 0)
 			(show_name no)
@@
 			)
 		)
-		(property "JLCPCB Part" "C25819"
+		(property "JLCPCB Part" "C4190"
 			(at 102.87 106.68 0)
 			(hide yes)
@@
 			)
 		)
-		(property "Manufacturer Part" "0603WAF4702T5E"
+		(property "Manufacturer Part" "0603WAF2201T5E"
 			(at 102.87 106.68 0)
 			(hide yes)
@@
 			)
 		)
-		(property "Value" "47K"
+		(property "Value" "2.2K"
 			(at 91.44 107.9499 0)
 			(show_name no)
@@
 			)
 		)
-		(property "JLCPCB Part" "C25819"
+		(property "JLCPCB Part" "C4190"
 			(at 93.98 106.68 0)
 			(hide yes)
@@
 			)
 		)
-		(property "Manufacturer Part" "0603WAF4702T5E"
+		(property "Manufacturer Part" "0603WAF2201T5E"
 			(at 93.98 106.68 0)
 			(hide yes)

Commit message: Initial software release
Added an initial sine generator application.
Only the I2S output is working via PIO.
Connections:
- net GND: now also U5.2 (XTI)
- no-connect marks 2 -> 1
Changed lines of the file:
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@@
 		(at 119.38 92.71)
 	)
-	(no_connect
-		(at 119.38 95.25)
-	)
 	(wire
 		(pts
@@
 	(wire
 		(pts
-			(xy 119.38 95.25) (xy 121.92 95.25)
+			(xy 119.38 92.71) (xy 121.92 92.71)
 		)
 		(stroke
@@
 	(wire
 		(pts
-			(xy 119.38 92.71) (xy 121.92 92.71)
+			(xy 166.37 50.8) (xy 166.37 52.07)
 		)
 		(stroke
@@
 	(wire
 		(pts
-			(xy 166.37 50.8) (xy 166.37 52.07)
+			(xy 157.48 69.85) (xy 167.64 69.85)
 		)
 		(stroke
@@
 	(wire
 		(pts
-			(xy 157.48 69.85) (xy 167.64 69.85)
+			(xy 166.37 59.69) (xy 166.37 60.96)
 		)
 		(stroke
@@
 	(wire
 		(pts
-			(xy 166.37 59.69) (xy 166.37 60.96)
+			(xy 137.16 133.35) (xy 137.16 135.89)
 		)
 		(stroke
@@
 	(wire
 		(pts
-			(xy 137.16 133.35) (xy 137.16 135.89)
+			(xy 154.94 115.57) (xy 152.4 115.57)
 		)
 		(stroke
@@
 	(wire
 		(pts
-			(xy 154.94 115.57) (xy 152.4 115.57)
+			(xy 115.57 60.96) (xy 115.57 59.69)
 		)
 		(stroke
@@
 	(wire
 		(pts
-			(xy 115.57 60.96) (xy 115.57 59.69)
+			(xy 116.84 90.17) (xy 114.3 90.17)
 		)
 		(stroke
@@
 	(wire
 		(pts
+			(xy 114.3 90.17) (xy 114.3 92.71)
+		)
+		(stroke
+			(width 0)
+			(type default)
+		)
+	)
+	(wire
+		(pts
 			(xy 154.94 105.41) (xy 152.4 105.41)
 		)
@@
 	(wire
 		(pts
+			(xy 116.84 95.25) (xy 116.84 90.17)
+		)
+		(stroke
+			(width 0)
+			(type default)
+		)
+	)
+	(wire
+		(pts
 			(xy 187.96 107.95) (xy 187.96 110.49)
 		)
@@
 	(wire
 		(pts
+			(xy 116.84 95.25) (xy 121.92 95.25)
+		)
+		(stroke
+			(width 0)
+			(type default)
+		)
+	)
+	(wire
+		(pts
 			(xy 167.64 69.85) (xy 167.64 71.12)
 		)
@@
 					(unit 1)
 				)
+			)
+		)
+	)
+	(symbol
+		(lib_id "power:GND")
+		(at 114.3 92.71 0)
+		(mirror y)
+		(unit 1)
+		(body_style 1)
+		(exclude_from_sim no)
+		(in_bom yes)
+		(on_board yes)
+		(in_pos_files yes)
+		(dnp no)
+		(fields_autoplaced yes)
+		(property "Reference" "#PWR065"
+			(at 114.3 99.06 0)
+			(hide yes)
+			(show_name no)
+			(do_not_autoplace no)
+			(effects
+				(font
+					(size 1.27 1.27)
+				)
+			)
+		)
+		(property "Value" "GND"
+			(at 114.3 97.79 0)
+			(show_name no)
+			(do_not_autoplace no)
+			(effects
+				(font
+					(size 1.27 1.27)
+				)
+			)
+		)
+		(property "Footprint" ""
+			(at 114.3 92.71 0)
+			(hide yes)
+			(show_name no)
+			(do_not_autoplace no)
+			(effects
+				(font
+					(size 1.27 1.27)
+				)
+			)
+		)
+		(property "Datasheet" ""
+			(at 114.3 92.71 0)
+			(hide yes)
+			(show_name no)
+			(do_not_autoplace no)
+			(effects
+				(font
+					(size 1.27 1.27)
+				)
+			)
+		)
+		(property "Description" "Power symbol creates a global label with name \"GND\" , ground"
+			(at 114.3 92.71 0)
+			(hide yes)
+			(show_name no)
+			(do_not_autoplace no)
+			(effects
+				(font
+					(size 1.27 1.27)
+				)
+			)
+		)
+		(pin "1"
+		)
+		(instances
+			(project "PicoFX"
+				(path "/4cbf131b-42e8-4a05-beea-68c6d66cdb1a/f7920eb9-f1f4-4882-8d74-32484732cce5"
+					(reference "#PWR065")
+					(unit 1)
+				)
