File: Hardware/PicoFX.kicad_pcb (KiCad board)
At the start: 4 copper layers, 59 x 95 mm, 102 parts, among them J1 RPI_ADC, J2 RP_GPIO, U1 AMS1117-5.0, U2 AMS1117-3.3, U3 MCP6002-xSN, U4 MCP6002-xSN, U5 CS4272, X1 PEDAL_COMBO_TOP

Commit message: Name update
Updated the name of the project.
Updated the silkscreen for the PCB layout.
Parts:
- moved G*** 0.98 mm to (169.4, 110.9)
- moved REF** 0.33 mm to (135.1, 118.3)
Other:
- board text added: "PICOFX GUITAR"
- board text removed: "SIMPLE CODEC"
