File: Hardware/PicoFX.kicad_pcb (KiCad board)
At the start: 4 copper layers, 59 x 95 mm, 102 parts, among them J1 RPI_ADC, J2 RP_GPIO, U1 AMS1117-5.0, U2 AMS1117-3.3, U3 MCP6002-xSN, U4 MCP6002-xSN, U5 CS4272, X1 PEDAL_COMBO_TOP

Commit message: Layout review
Updated the LDO layout to include a series resistor for stability.
Updated all build files.
Parts:
- removed the C14 at (122.8, 102.4)
- removed the C6 at (147.6, 75.6)
- added C13: 10u, Capacitor_SMD:C_0805_2012Metric, B.Cu at (135.2, 100.4)
- added C7: 10u, Capacitor_SMD:C_0805_2012Metric, B.Cu at (148.2, 78.4)
- added R3: 1, Resistor_SMD:R_0603_1608Metric, B.Cu at (147.6, 75.4)
- added R4: 1, Resistor_SMD:R_0603_1608Metric, B.Cu at (135.2, 103.0)
- moved C10 2.00 mm to (122.8, 100.4), turned to -90 degrees
- renumbered C11 to C10, C10 to C11, C13 to C14, C7 to C6, C9 to C8, C8 to C9, R8 to R10, R9 to R11, R10 to R12, R11 to R13, R12 to R14, R13 to R15, R14 to R16, R15 to R17, R16 to R18, R17 to R19, R18 to R20, R19 to R21, R20 to R22, R21 to R23, R22 to R24, R23 to R25, R24 to R26, R25 to R27, R26 to R28, R27 to R29, R28 to R30, R29 to R31, R30 to R32, R3 to R5, R4 to R6, R5 to R7, R6 to R8, R7 to R9
Routing:
- net Net-(C7-Pad1): track 0.00 -> 2.32 mm
- net Net-(C13-Pad1): track 0.00 -> 2.08 mm
- net +3V3D: track 171.3 -> 169.4 mm
- net GND: track 23.2 -> 24.2 mm, vias 288 -> 287

Commit message: Output files
Updated the board silkscreen.
Upddated the output files.
Parts:
- added G***: LOGO, Logos:Querub, F.Cu at (150.0, 79.8)
- moved R4 10.0 mm to (125.4, 105.2)
- moved C13 10.0 mm to (125.4, 102.4), turned to -90 degrees
- moved FB2 6.20 mm to (130.6, 93.2)
- moved C10 3.28 mm to (125.4, 98.4), turned to 90 degrees
- moved R3 3.09 mm to (148.3, 78.4), turned to 0 degrees
- moved C7 3.06 mm to (147.6, 75.4), turned to -90 degrees
- moved U2 2.60 mm to (131.6, 100.4)
- moved G*** 1.85 mm to (169.4, 112.7)
- moved C6 0.60 mm to (127.8, 91.8), turned to 180 degrees
- moved C8 0.60 mm to (127.8, 94.6), turned to 180 degrees
Connections:
- C13 pad 1: Net-(C13-Pad1) -> +3V3D
- C13 pad 2: GND -> Net-(C13-Pad2)
- C7 pad 1: Net-(C7-Pad1) -> +5VA_RAW
- C7 pad 2: GND -> Net-(C7-Pad2)
- R3 pad 1: +5VA_RAW -> Net-(C7-Pad2)
- R3 pad 2: Net-(C7-Pad1) -> GND
- R4 pad 1: +3V3D -> Net-(C13-Pad2)
- R4 pad 2: Net-(C13-Pad1) -> GND
Routing:
- net +3V3D: track 169.4 -> 171.8 mm
- net Net-(C7-Pad1): track 2.32 -> 0.00 mm
- net Net-(C13-Pad2): track 0.00 -> 2.28 mm
- net Net-(C7-Pad2): track 0.00 -> 2.09 mm
- net Net-(C13-Pad1): track 2.08 -> 0.00 mm
- net +VCC: track 59.9 -> 61.2 mm
- net GND: track 24.2 -> 24.0 mm, vias 287 -> 283
